Commit message: Update pioneer3dx.xacro
Moving the lms100 sensor to a lower position

File: p3dx_description/urdf/pioneer3dx.xacro (robot description, xacro)
@@ -212,5 +212,5 @@
 	<joint name="lms100_joint" type="fixed">
 		<axis xyz="0 1 0" />
-		<origin xyz="0.12 0 0.26" rpy="0 0 0" />
+		<origin xyz="0.15 0 0.08" rpy="0 0 0" />
 		<parent link="base_link" />
 		<child link="lms100" />
